File: current_shunt.kicad_pcb (KiCad board)
At the start: 2 copper layers, 82 x 72 mm, 20 parts, among them J1 Conn_01x01, J10 Conn_01x01, J11 Conn_01x01, J12 Conn_01x01, J13 Conn_01x01, J2 Conn_01x01, J3 Conn_01x01, J4 Conn_01x01, J6 Conn_01x01, J8 Conn_01x01

Commit message: Cleanups and fixes
Parts:
- moved J11 6.73 mm to (171.0, 105.5)
- moved J13 6.07 mm to (141.0, 101.0)
Routing:
- net GND: track 38.6 -> 48.1 mm
- net Net-(J8-Pad1): track 7.38 -> 10.2 mm
- net Net-(J6-Pad1): track 7.38 -> 9.27 mm
- net Net-(J3-Pad1): track 9.99 -> 11.8 mm
- net Net-(J10-Pad1): track 4.00 -> 4.91 mm
