File: current_shunt.kicad_sch (KiCad schematic)
At the start: 20 parts, among them J1 Conn_01x01, J10 Conn_01x01, J11 Conn_01x01, J12 Conn_01x01, J13 Conn_01x01, J2 Conn_01x01, J3 Conn_01x01, J4 Conn_01x01, J6 Conn_01x01, J8 Conn_01x01

Commit message: Fix part number
Parts:
- R5: AVL P/N MFR03SF100KA10 -> MFR03SF100JA10; LCSC C113667 -> C58751
Changed lines of the file:
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@@
       (effects (font (size 1.27 1.27)) hide)
     )
-    (property "AVL P/N" "MFR03SF100KA10" (id 5) (at 93.98 147.32 0)
+    (property "AVL P/N" "MFR03SF100JA10" (id 5) (at 93.98 147.32 0)
       (effects (font (size 1.27 1.27)) hide)
     )
-    (property "LCSC" "C113667" (id 6) (at 93.98 147.32 0)
+    (property "LCSC" "C58751" (id 6) (at 93.98 147.32 0)
       (effects (font (size 1.27 1.27)) hide)
     )
